File: PCB/92pi/92pi.kicad_sch (KiCad schematic)
At the start: 0 parts

Commit message: some stuff
Parts:
- added C12, C13: 10uF, Capacitor_SMD:C_0603_1608Metric, symbol Device:C_Small
- added C14: 10uF, Capacitor_SMD:C_0603_1608Metric, symbol Device:C
- added C15: 100nF, Capacitor_SMD:C_0603_1608Metric, symbol Device:C
- added C16: 22uF, Capacitor_SMD:C_1206_3216Metric, symbol Device:C
- added C17, C18: 100uF, Capacitor_Tantalum_SMD:CP_EIA-3528-15_AVX-H, symbol Device:C_Polarized
- added D19: D_Schottky_Small, Diode_SMD:D_SOD-323, symbol Device:D_Schottky_Small
- added D29: Notification LED, _mod_files:FM-B2020RGBA-HG, symbol Device:LED_RBAG
- added D82: B5819W, Diode_SMD:D_SOD-123, symbol Device:D_Schottky
- added J1: USB_B, _mod_files:UJ2BH2TH, symbol Connector:USB_B
- added J2: Battery, Connector_JST:JST_PH_S2B-PH-SM4-TB_1x02-1MP_P2.00mm_Horizontal, symbol Connector:Conn_01x02_Male
- added J3: PROG, Connector_PinSocket_2.54mm:PinSocket_2x04_P2.54mm_Horizontal, symbol Connector_Generic:Conn_02x04_Odd_Even
- added JP1: PC_PWR_FORCE, Jumper:SolderJumper-2_P1.3mm_Open_RoundedPad1.0x1.5mm, symbol Jumper:Jumper_2_Open
- added JP2: USB_ONLY, Jumper:SolderJumper-2_P1.3mm_Open_RoundedPad1.0x1.5mm, symbol Jumper:Jumper_2_Open
- added KB_INT1, KB_SCL1, KB_SDA1, TB_GND1, TP_3.3: TestPoint, TestPoint:TestPoint_Pad_D1.0mm, symbol Connector:TestPoint
- added L1: 6.8uH/4A, Inductor_SMD:L_Bourns_SRP7028A_7.3x6.6mm, symbol Device:L
- added Q1: SI2301, Package_TO_SOT_SMD:SOT-23, symbol Transistor_FET:FDN340P
- added Q2: SI2301, Package_TO_SOT_SMD:SOT-23, symbol Transistor_FET:DMG2301L
- added Q3: S8050, Package_TO_SOT_SMD:SOT-23, symbol Device:Q_NPN_BEC
- added R10, R11: 100K, Resistor_SMD:R_0603_1608Metric, symbol Device:R_Small
- added R12: 220, Resistor_SMD:R_0603_1608Metric, symbol Device:R
- added R13, R14: 100, Resistor_SMD:R_0603_1608Metric, symbol Device:R
- added R15, R16, R25: 10K, Resistor_SMD:R_0603_1608Metric, symbol Device:R
- added R17, R20: 100K, Resistor_SMD:R_0603_1608Metric, symbol Device:R
- added R18, R22: 2M, Resistor_SMD:R_0603_1608Metric, symbol Device:R
- added R19: 360K, Resistor_SMD:R_0603_1608Metric, symbol Device:R
- added R21: 1M, Resistor_SMD:R_0603_1608Metric, symbol Device:R
- added R23: 220K, Resistor_SMD:R_0603_1608Metric, symbol Device:R
- added R24: 330, Resistor_SMD:R_0603_1608Metric, symbol Device:R
- added SW1: ON/OFF, Button_Switch_SMD:SW_SPDT_PCM12, symbol Switch:SW_SPST
- added U2: AP2112K-3.3, Package_TO_SOT_SMD:SOT-23-5, symbol Regulator_Linear:AP2112K-3.3
- added U5: TP4054, Package_TO_SOT_SMD:SOT-23-5, symbol Battery_Management:MCP73831-2-OT
- added U6: TPS61090, Package_SO:HTSSOP-16-1EP_4.4x5mm_P0.65mm_EP3.4x5mm_Mask2.46x2.31mm_ThermalVias, symbol beepy:TPS61090
Connections:
- new net: C14.1, C15.1, D82.1 (K), L1.1, Q1.2 (S), R18.1, SW1.1 (A), U6.6 (VBAT)
- new net: R16.2, U5.5 (PROG)
- new net: R20.2, SW1.2 (B), U6.9 (EN)
- new net: D29.4 (GK), R13.2
- new net: D29.1 (RK), R12.2
- new net: Q2.1 (G), Q3.3 (C), R15.2
- new net: L1.2, U6.1 (SW), U6.2 (SW)
- new net: R22.2, R23.1, U6.12 (FB)
- new net: R18.2, R19.1, U6.7 (LBI)
- new net: Q3.1 (B), R24.2
- new net: D29.2 (BK), R14.2
- new net +3.3V: TP_3.3.1
- new net +3V3: C13.2, D19.2 (A), D29.3 (A), J3.6 (Pin_6), R21.2, U2.5 (VOUT)
- new net +5V: C12.1, C16.1, C17.1, C18.1, D19.1 (K), J3.8 (Pin_8), JP1.1 (A), JP2.2 (B), Q2.2 (S), R15.1, R22.1, U2.1 (VIN), U2.3 (EN), U6.13 (VOUT), U6.14 (VOUT), U6.15 (VOUT)
- new net +BATT: J2.1 (Pin_1), Q1.3 (D), R10.1, U5.3 (VBAT)
- new net BOOTSEL: J3.1 (Pin_1)
- new net GND: C12.2, C13.1, C14.2, C15.2, C16.2, C17.2, C18.2, J1.4 (GND), J2.2 (Pin_2), J3.2 (Pin_2), J3.4 (Pin_4), Q3.2 (E), R11.2, R16.1, R17.2, R19.2, R20.1, R23.2, R25.1, TB_GND1.1, U2.2 (GND), U5.2 (VSS), U6.11 (GND), U6.17 (PAD), U6.3 (PGND), U6.4 (PGND), U6.5 (PGND), U6.8 (SYNC)
- new net Keyboard/BATT_ADC: R10.2, R11.1
- new net Keyboard/KB_INT: KB_INT1.1
- new net Keyboard/KB_SCL: KB_SCL1.1
- new net Keyboard/KB_SDA: KB_SDA1.1
- new net Keyboard/LED_B: R14.1
- new net Keyboard/LED_G: R13.1
- new net Keyboard/LED_R: R12.1
- new net LBO: R21.1, U6.10 (LBO)
- new net PC_PWR_5v: JP1.2 (B), Q2.3 (D)
- new net PC_PWR_ENABLE: R24.1, R25.2
- new net USB_D+: J1.3 (D+)
- new net USB_D-: J1.2 (D-)
- new net VBUS: D82.2 (A), J1.1 (VBUS), JP2.1 (A), Q1.1 (G), R17.1, U5.4 (VDD)
- new net ~{RESET}: J3.3 (Pin_3)
- no-connect marks 0 -> 1
Other:
- sheet Keyboard ports: added BATT_ADC, KB_INT, KB_SCL, KB_SDA, LED_B, LED_G, LED_R; removed none
- note added: "OPT: Battery Charging FOR USE WITH USB ONLY, SOLDER JUMPER"

Commit message: stuff did
Connections:
- net +3.3V is gone; now on net +3V3: TP_3.3.1
Other:
- sheet Keyboard ports: added +3.3; removed none
- moved on the sheet: TP_3.3
Changed lines of the file:
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@@
   (junction (at 99.822 46.101) (diameter 0) (color 0 0 0 0)
+  )
+  (junction (at 231.14 57.15) (diameter 0) (color 0 0 0 0)
   )
   (junction (at 79.502 46.101) (diameter 0) (color 0 0 0 0)
@@
     (stroke (width 0) (type default))
   )
+  (wire (pts (xy 231.14 55.88) (xy 231.14 57.15))
+    (stroke (width 0) (type default))
+  )
   (wire (pts (xy 154.94 118.745) (xy 153.67 118.745))
     (stroke (width 0) (type solid))
@@
     (stroke (width 0) (type solid))
   )
+  (wire (pts (xy 227.33 57.15) (xy 231.14 57.15))
+    (stroke (width 0) (type default))
+  )
   (wire (pts (xy 69.342 46.101) (xy 79.502 46.101))
     (stroke (width 0) (type default))
@@
   )
   (wire (pts (xy 213.36 69.215) (xy 213.36 70.485))
+    (stroke (width 0) (type default))
+  )
+  (wire (pts (xy 231.14 57.15) (xy 231.14 59.69))
     (stroke (width 0) (type default))
   )
@@
     (effects (font (size 1.27 1.27)) (justify left bottom))
   )
-  (label "LBO" (at 107.95 166.37 180) (fields_autoplaced)
+  (label "LBO" (at 102.87 158.115 180) (fields_autoplaced)
     (effects (font (size 1.27 1.27)) (justify right bottom))
   )
@@
     )
   )
-  (symbol (lib_id "Connector:TestPoint") (at 205.105 69.215 0) (unit 1)
-    (in_bom yes) (on_board yes) (dnp no)
-    (property "Reference" "TP_3.3" (at 205.105 53.975 90)
-      (effects (font (size 1.27 1.27)) (justify left))
-    )
-    (property "Value" "TestPoint" (at 205.105 64.135 90)
-      (effects (font (size 1.27 1.27)) (justify left))
-    )
-    (property "Footprint" "TestPoint:TestPoint_Pad_D1.0mm" (at 210.185 69.215 0)
-      (effects (font (size 1.27 1.27)) hide)
-    )
-    (property "Datasheet" "~" (at 210.185 69.215 0)
+  (symbol (lib_id "Connector:TestPoint") (at 227.33 57.15 0) (unit 1)
+    (in_bom yes) (on_board yes) (dnp no)
+    (property "Reference" "TP_3.3" (at 227.33 41.91 90)
+      (effects (font (size 1.27 1.27)) (justify left))
+    )
+    (property "Value" "TestPoint" (at 227.33 52.07 90)
+      (effects (font (size 1.27 1.27)) (justify left))
+    )
+    (property "Footprint" "TestPoint:TestPoint_Pad_D1.0mm" (at 232.41 57.15 0)
+      (effects (font (size 1.27 1.27)) hide)
+    )
+    (property "Datasheet" "~" (at 232.41 57.15 0)
       (effects (font (size 1.27 1.27)) hide)
     )
@@
     )
   )
+  (symbol (lib_id "power:+3.3V") (at 231.14 55.88 0) (mirror y) (unit 1)
+    (in_bom yes) (on_board yes) (dnp no)
+    (property "Reference" "#PWR061" (at 231.14 59.69 0)
+      (effects (font (size 1.27 1.27)) hide)
+    )
+    (property "Value" "+3.3V" (at 231.14 52.07 0)
+      (effects (font (size 1.27 1.27)))
+    )
+    (property "Footprint" "" (at 231.14 55.88 0)
+      (effects (font (size 1.27 1.27)) hide)
+    )
+    (property "Datasheet" "" (at 231.14 55.88 0)
+      (effects (font (size 1.27 1.27)) hide)
+    )
+    (pin "1")
+    (instances
+      (project "92pi"
+        (path "/6de8b922-75ab-426d-b031-f6a8fb5afbd4"
+          (reference "#PWR061") (unit 1)
+        )
+      )
+      (project "beepy"
+        (path "/e63e39d7-6ac0-4ffd-8aa3-1841a4541b55/832ef58d-0dd2-4973-9055-9966f4d0abfc"
+          (reference "#PWR0107") (unit 1)
+        )
+      )
+    )
+  )
   (symbol (lib_id "Device:C_Polarized") (at 162.56 88.9 0) (unit 1)
     (in_bom yes) (on_board yes) (dnp no) (fields_autoplaced)
@@
         (path "/6de8b922-75ab-426d-b031-f6a8fb5afbd4"
           (reference "KB_INT1") (unit 1)
-        )
-      )
-    )
-  )
-  (symbol (lib_name "+3.3V_1") (lib_id "power:+3.3V") (at 205.105 69.215 180) (unit 1)
-    (in_bom yes) (on_board yes) (dnp no)
-    (property "Reference" "#PWR058" (at 205.105 65.405 0)
-      (effects (font (size 1.27 1.27)) hide)
-    )
-    (property "Value" "+3.3V" (at 205.105 74.93 90)
-      (effects (font (size 1.27 1.27)))
-    )
-    (property "Footprint" "" (at 205.105 69.215 0)
-      (effects (font (size 1.27 1.27)) hide)
-    )
-    (property "Datasheet" "" (at 205.105 69.215 0)
-      (effects (font (size 1.27 1.27)) hide)
-    )
-    (pin "1")
-    (instances
-      (project "92pi"
-        (path "/6de8b922-75ab-426d-b031-f6a8fb5afbd4"
-          (reference "#PWR058") (unit 1)
         )
       )
@@
       (effects (font (size 1.27 1.27)) (justify right))
     )
+    (pin "+3.3" input (at 231.14 59.69 90)
+      (effects (font (size 1.27 1.27)) (justify right))
+    )
