File: PCB/92pi/keyboard.kicad_sch (KiCad schematic)
At the start: 94 parts

Commit message: kinda?
Parts:
- removed D?: 1N4148, Diode_THT:D_DO-35_SOD27_P7.62mm_Horizontal, symbol Diode:1N4148
- removed SW? (x86): (no value), symbol Switch:SW_Push_45deg
- added D? (x85): 1N914WT, Diode_SMD:D_SOD-523, symbol Diode:1N914WT
- added R? (x2): R27, symbol Device:R
- added SW? (x85): SW_SPST, symbol Switch:SW_SPST
- added TP?: USB_DP, symbol Connector:TestPoint
- added TP?: USB_DM, symbol Connector:TestPoint
Connections:
- net +3.3V: now also U?.48 (USB_VDD)
- net Row 0: now also D?.1 (K)
- net Row 1: now also D?.1 (K)
- net Row 2: now also D?.1 (K)
- net Row 3: now also D?.1 (K)
- net Row 4: now also D?.1 (K)
- net +1V1: now reaches U?.23 (DVDD), U?.50 (DVDD)
- net +1V1: now also U?.45 (VREG_VOUT)
- net at U?.46 (USB_DM): now also R?.2
- net at U?.47 (USB_DP): now also R?.2
- new net: D?.2 (A), SW?.1 (A) (x85)
- new net USB_DM: R?.1, TP?.1
- new net USB_DP: R?.1, TP?.1
Other:
- note added: "5x17 matrix for 85 keys"
- moved on the sheet: R?, SW?

Commit message: keyboards kinda how i want i think
Parts:
- removed D? (x4): 1N914WT, Diode_SMD:D_SOD-523, symbol Diode:1N914WT
- removed SW? (x4): SW_SPST, symbol Switch:SW_SPST
- SW?: value SW_SPST -> SW_F4
- SW?: value SW_SPST -> SW_NP2
- SW?: value SW_SPST -> SW_CLOSE_PAREN
- SW?: value SW_SPST -> SW_F3
- SW?: value SW_SPST -> SW_CLEAR
- SW?: value SW_SPST -> SW_F6
- SW?: value SW_SPST -> SW_N
- SW?: value SW_SPST -> SW_COS
- SW?: value SW_SPST -> SW_NP8
- SW?: value SW_SPST -> SW_Y
- SW?: value SW_SPST -> SW_O
- SW?: value SW_SPST -> SW_LN
- SW?: value SW_SPST -> SW_J
- SW?: value SW_SPST -> SW_CAMA
- SW?: value SW_SPST -> SW_SIN
- SW?: value SW_SPST -> SW_DP_UP
- SW?: value SW_SPST -> SW_KB_ENTER
- SW?: value SW_SPST -> SW_=
- SW?: value SW_SPST -> SW_X
- SW?: value SW_SPST -> SW_NP.
- SW?: value SW_SPST -> SW_K
- SW?: value SW_SPST -> SW_ESC
- SW?: value SW_SPST -> SW_GREEN_STAR
- SW?: value SW_SPST -> SW_RIGHT_2ND
- SW?: value SW_SPST -> SW_NP+
- SW?: value SW_SPST -> SW_GP_ENTER
- SW?: value SW_SPST -> SW_F
- SW?: value SW_SPST -> SW_NP9
- SW?: value SW_SPST -> SW_F2
- SW?: value SW_SPST -> SW_SEMICOLEN
- SW?: value SW_SPST -> SW_Q
- SW?: value SW_SPST -> SW_A
- SW?: value SW_SPST -> SW_NP_ENT
- SW?: value SW_SPST -> SW_APPS
- SW?: value SW_SPST -> SW_LEFT_2ND
- SW?: value SW_SPST -> SW_L
- SW?: value SW_SPST -> SW_T
- SW?: value SW_SPST -> SW_U
- SW?: value SW_SPST -> SW_DP_DOWN
- SW?: value SW_SPST -> SW_TAN
- SW?: value SW_SPST -> SW_P
- SW?: value SW_SPST -> SW_NP1
- SW?: value SW_SPST -> SW_G
- SW?: value SW_SPST -> SW_C
- SW?: value SW_SPST -> SW_NP0
- SW?: value SW_SPST -> SW_LCKHND
- SW?: value SW_SPST -> SW_STO
- SW?: value SW_SPST -> SW_SPACE
- SW?: value SW_SPST -> SW_S
- SW?: value SW_SPST -> SW_NP7
- SW?: value SW_SPST -> SW_Z
- SW?: value SW_SPST -> SW_SHIFT
- SW?: value SW_SPST -> SW_R
- SW?: value SW_SPST -> SW_DIV
- SW?: value SW_SPST -> SW_NP*
- SW?: value SW_SPST -> SW_GP_ENTER_0
- SW?: value SW_SPST -> SW_V
- SW?: value SW_SPST -> SW_BACKSPACE
- SW?: value SW_SPST -> SW_F5
- SW?: value SW_SPST -> SW_F1
- SW?: value SW_SPST -> SW_DP_LEFT
- SW?: value SW_SPST -> SW_NP(-)
- SW?: value SW_SPST -> SW_F7
- SW?: value SW_SPST -> SW_I
- SW?: value SW_SPST -> SW_POW
- SW?: value SW_SPST -> SW_NP5
- SW?: value SW_SPST -> SW_H
- SW?: value SW_SPST -> SW_W
- SW?: value SW_SPST -> SW_NP3
- SW?: value SW_SPST -> SW_F8
- SW?: value SW_SPST -> SW_MODE
- SW?: value SW_SPST -> SW_OPEN_PAREN
- SW?: value SW_SPST -> SW_B
- SW?: value SW_SPST -> SW_NP4
- SW?: value SW_SPST -> SW_M
- SW?: value SW_SPST -> SW_RIGHT
- SW?: value SW_SPST -> SW_NP-
- SW?: value SW_SPST -> SW_NP6
- SW?: value SW_SPST -> SW_GP_ENTER_1
- SW?: value SW_SPST -> SW_D
- SW?: value SW_SPST -> SW_E
Connections:
- net Row 5 is gone; now on net Row 2: U?.30 (GPIO19)
- net Row 6 is gone; now on net Row 3: U?.31 (GPIO20)
- net Row 7 is gone; now on net Row 4: U?.32 (GPIO21)
- net Col 0: now also SW?.2 (B), SW?.2 (B), SW?.2 (B), SW?.2 (B)
- net Col 1: now also SW?.2 (B), SW?.2 (B), SW?.2 (B), SW?.2 (B), SW?.2 (B)
- net Col 10: now also SW?.2 (B), SW?.2 (B), SW?.2 (B), SW?.2 (B), SW?.2 (B)
- net Col 11: now also SW?.2 (B), SW?.2 (B), SW?.2 (B), SW?.2 (B), SW?.2 (B)
- net Col 12: now also SW?.2 (B), SW?.2 (B), SW?.2 (B), SW?.2 (B), SW?.2 (B)
- net Col 13: now also SW?.2 (B), SW?.2 (B), SW?.2 (B), SW?.2 (B), SW?.2 (B)
- net Col 2: now also SW?.2 (B), SW?.2 (B), SW?.2 (B)
- net Col 3: now also SW?.2 (B), SW?.2 (B), SW?.2 (B), SW?.2 (B)
- net Col 4: now also SW?.2 (B), SW?.2 (B), SW?.2 (B), SW?.2 (B), SW?.2 (B)
- net Col 5: now also SW?.2 (B), SW?.2 (B), SW?.2 (B), SW?.2 (B), SW?.2 (B)
- net Col 6: now also SW?.2 (B), SW?.2 (B), SW?.2 (B), SW?.2 (B), SW?.2 (B)
- net Col 7: now also SW?.2 (B), SW?.2 (B), SW?.2 (B), SW?.2 (B), SW?.2 (B)
- net Col 8: now also SW?.2 (B), SW?.2 (B), SW?.2 (B), SW?.2 (B), SW?.2 (B)
- net Col 9: now also SW?.2 (B), SW?.2 (B), SW?.2 (B), SW?.2 (B), SW?.2 (B)
- net Row 0: now also D?.1 (K), D?.1 (K), D?.1 (K), D?.1 (K), D?.1 (K), D?.1 (K), D?.1 (K), D?.1 (K), D?.1 (K), D?.1 (K), D?.1 (K), D?.1 (K), D?.1 (K), D?.1 (K), D?.1 (K), D?.1 (K), U?.28 (GPIO17); no longer U?.17 (GPIO14)
- net Row 1: now also D?.1 (K), D?.1 (K), D?.1 (K), D?.1 (K), D?.1 (K), D?.1 (K), D?.1 (K), D?.1 (K), D?.1 (K), D?.1 (K), D?.1 (K), D?.1 (K), D?.1 (K), D?.1 (K), D?.1 (K), D?.1 (K), U?.29 (GPIO18); no longer U?.18 (GPIO15)
- net Row 2: now also D?.1 (K), D?.1 (K), D?.1 (K), D?.1 (K), D?.1 (K), D?.1 (K), D?.1 (K), D?.1 (K), D?.1 (K), D?.1 (K), D?.1 (K), D?.1 (K), D?.1 (K), D?.1 (K), D?.1 (K); no longer U?.27 (GPIO16)
- net Row 3: now also D?.1 (K), D?.1 (K), D?.1 (K), D?.1 (K), D?.1 (K), D?.1 (K), D?.1 (K), D?.1 (K), D?.1 (K), D?.1 (K), D?.1 (K), D?.1 (K), D?.1 (K), D?.1 (K); no longer U?.28 (GPIO17)
- net Row 4: now also D?.1 (K), D?.1 (K), D?.1 (K), D?.1 (K), D?.1 (K), D?.1 (K), D?.1 (K), D?.1 (K), D?.1 (K), D?.1 (K), D?.1 (K), D?.1 (K), D?.1 (K), D?.1 (K), D?.1 (K), D?.1 (K); no longer U?.29 (GPIO18)
- net Col 14: now reaches SW?.2 (B)
- net Col 14: now also SW?.2 (B), SW?.2 (B), SW?.2 (B), SW?.2 (B), U?.17 (GPIO14)
- net Col 16: now reaches SW?.2 (B)
- net Col 16: now also SW?.2 (B), SW?.2 (B), SW?.2 (B), SW?.2 (B), U?.27 (GPIO16)
- net Col 15: now reaches SW?.2 (B)
- net Col 15: now also SW?.2 (B), SW?.2 (B), SW?.2 (B), SW?.2 (B), U?.18 (GPIO15)
- net Row 8: no longer names the net of U?.34 (GPIO22)
Other:
- note added: "Make sure this is really 27 ohms and that i didnt do something silly copying the scmatic >.<"
- note added: "TODO: On the next schmatic up, Split the USB and have a Switch so that it can go into a PC or into the SOC"

Commit message: some stuff
Parts:
- removed C? (x2): 27p, symbol Device:C_Small
- removed D? (x2): 1N914WT, Diode_SMD:D_SOD-523, symbol Diode:1N914WT
- removed R?: R1K, symbol Device:R
- removed R? (x2): R27, symbol Device:R
- removed R?: R100k, symbol Device:R
- removed SW?: SW_GP_ENTER, symbol Switch:SW_SPST
- removed SW?: SW_SPST, symbol Switch:SW_SPST
- removed SW?: SW_GP_ENTER_1, symbol Switch:SW_SPST
- removed TP?: USB_DP, symbol Connector:TestPoint
- removed TP?: USB_DM, symbol Connector:TestPoint
- removed U?: RP2040, Package_DFN_QFN:QFN-56-1EP_7x7mm_P0.4mm_EP3.2x3.2mm, symbol MCU_RaspberryPi:RP2040
- removed Y?: ABLS-12.00MHZ-B4-T, symbol Device:Crystal
- added C1, C2: 12pF, Capacitor_SMD:C_0603_1608Metric, symbol Device:C_Small
- added C10, C3, C4, C5, C6, C7, C9: 0.1uF, Capacitor_SMD:C_0603_1608Metric, symbol Device:C_Small
- added C11, C8: 1uF, Capacitor_SMD:C_0603_1608Metric, symbol Device:C_Small
- added R1, R2: 27R, Resistor_SMD:R_0603_1608Metric, symbol Device:R_Small
- added R3, R5: 1K, Resistor_SMD:R_0603_1608Metric, symbol Device:R_Small
- added R4, R6, R9: 10K, Resistor_SMD:R_0603_1608Metric, symbol Device:R_Small
- added R7, R8: 4.7K, Resistor_SMD:R_0603_1608Metric, symbol Device:R_Small
- added U1: RP2040, _mod_files:QFN-56-1EP_7x7mm_P0.4mm_EP5.6x5.6mm, symbol MCU_RaspberryPi:RP2040
- added U3: GD25Q16xS, Package_SO:SSOP-8_5.25x5.24mm_P1.27mm, symbol Memory_Flash_Extra:W25Q64JV
- added Y1: XYDBPCNANF-12MHZ, Crystal:Crystal_SMD_3225-4Pin_3.2x2.5mm, symbol Device:Crystal_GND24_Small
- SW10, SW11, SW12, SW13, SW14, SW15, SW16, SW17, SW18, SW19, SW2, SW21, SW22, SW23, SW24, SW25, SW26, SW27, SW28, SW29, SW3, SW31, SW32, SW33, SW34, SW35, SW36, SW37, SW38, SW39, SW4, SW40, SW41, SW42, SW43, SW44, SW45, SW46, SW47, SW48, SW49, SW5, SW50, SW51, SW52, SW53, SW54, SW55, SW56, SW57, SW58, SW59, SW6, SW60, SW61, SW62, SW63, SW64, SW65, SW66, SW67, SW68, SW69, SW7, SW70, SW71, SW72, SW73, SW74, SW75, SW76, SW77, SW78, SW79, SW8, SW80, SW81, SW82, SW9: renamed from SW?; footprint (none) -> ModFiles:Kbpad
- gave numbers to parts that had none: 79
Connections:
- net Col 0: now also U1.2 (GPIO0)
- net Col 1: now also U1.3 (GPIO1)
- net Col 10: now also U1.13 (GPIO10)
- net Col 11: now also U1.14 (GPIO11)
- net Col 12: now also U1.15 (GPIO12)
- net Col 13: now also U1.16 (GPIO13)
- net Col 14: now also U1.17 (GPIO14)
- net Col 15: now also U1.18 (GPIO15)
- net Col 16: now also U1.27 (GPIO16)
- net Col 2: now also U1.4 (GPIO2)
- net Col 3: now also U1.5 (GPIO3)
- net Col 4: now also U1.6 (GPIO4)
- net Col 5: now also U1.7 (GPIO5)
- net Col 6: now also U1.8 (GPIO6)
- net Col 7: now also U1.9 (GPIO7)
- net Col 8: now also U1.11 (GPIO8)
- net Col 9: now also U1.12 (GPIO9)
- net GND: now also C1.2, C10.2, C11.2, C2.2, C3.2, C4.2, C5.2, C6.2, C7.2, C8.2, C9.2, U1.19 (TESTEN), U1.57 (GND), U3.4 (GND), U3.9 (GND), Y1.2, Y1.4
- net Row 0: now also U1.28 (GPIO17)
- net Row 1: now also U1.29 (GPIO18)
- net Row 2: now also U1.30 (GPIO19)
- net Row 3: now also U1.31 (GPIO20)
- net Row 4: now also U1.32 (GPIO21)
- new net: C2.1, R3.2, Y1.1
- new net: C1.1, U1.20 (XIN), Y1.3
- new net: R3.1, U1.21 (XOUT)
- new net: C10.1, C11.1, C9.1, U1.23 (DVDD), U1.45 (VREG_VOUT), U1.50 (DVDD)
- new net +3V3: C3.1, C4.1, C5.1, C6.1, C7.1, C8.1, R4.1, R6.2, R7.2, R8.1, R9.1, U1.1 (IOVDD), U1.10 (IOVDD), U1.22 (IOVDD), U1.33 (IOVDD), U1.42 (IOVDD), U1.43 (ADC_AVDD), U1.44 (VREG_VIN), U1.48 (USB_VDD), U1.49 (IOVDD), U3.8 (VDD)
- new net BATT_ADC: U1.38 (GPIO26)
- new net BOOTSEL: R5.1
- new net D+: R2.1, U1.47 (USB_D+)
- new net D-: R1.1, U1.46 (USB_D-)
- new net KB_INT: R9.2
- new net KB_SCL: R8.2, U1.41 (GPIO29)
- new net KB_SDA: R7.1, U1.40 (GPIO28)
- new net LED_B: U1.35 (GPIO23)
- new net LED_G: U1.36 (GPIO24)
- new net LED_R: U1.37 (GPIO25)
- new net QSPI_SCLK: U1.52 (QSPI_SCLK), U3.6 (SCK)
- new net QSPI_SD0: U1.53 (QSPI_SD0), U3.5 (DI/IO0)
- new net QSPI_SD1: U1.55 (QSPI_SD1), U3.2 (DO/IO1)
- new net QSPI_SD2: U1.54 (QSPI_SD2), U3.3 (~WP~/IO2)
- new net QSPI_SD3: U1.51 (QSPI_SD3), U3.7 (~HOLD~/IO3)
- new net SWCLK: U1.24 (SWCLK)
- new net SWDIO: U1.25 (SWDIO)
- new net USB_D+: R2.2
- new net USB_D-: R1.2
- new net ~{QSPI_CS}: R5.2, R6.1, U1.56 (~{QSPI_CS}), U3.1 (~CS~)
- new net ~{RESET}: R4.2, U1.26 (RUN)
- no-connect marks 0 -> 2
Other:
- note added: "10"
- note added: "12MHz"
- note added: "22"
- note added: "33"
- note added: "42"
- note added: "43"
- note added: "48"
- note added: "49"
- note added: "50"
- note added: "ADC"
- note added: "I2C0"
- note removed: "Make sure this is really 27 ohms and that i didnt do something silly copying the scmatic >.<"
- note removed: "TODO: On the next schmatic up, Split the USB and have a Switch so that it can go into a PC or into the SOC"

Commit message: .
Parts:
- SW10, SW11, SW12, SW13, SW14, SW15, SW16, SW17, SW18, SW19, SW2, SW21, SW22, SW23, SW24, SW25, SW26, SW27, SW28, SW29, SW3, SW31, SW32, SW33, SW34, SW35, SW36, SW37, SW38, SW39, SW4, SW40, SW41, SW42, SW43, SW44, SW45, SW46, SW47, SW48, SW49, SW5, SW50, SW51, SW52, SW53, SW54, SW55, SW56, SW57, SW58, SW59, SW6, SW60, SW61, SW62, SW63, SW64, SW65, SW66, SW67, SW68, SW69, SW7, SW70, SW71, SW72, SW73, SW74, SW75, SW76, SW77, SW78, SW79, SW8, SW80, SW81, SW82, SW9: footprint ModFiles:Kbpad -> mod_files:Kbpad

Commit message: stuff did
Changed lines of the file:
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@@
     (stroke (width 0) (type solid))
+  )
+  (wire (pts (xy 477.52 248.285) (xy 481.965 248.285))
+    (stroke (width 0) (type default))
   )
   (wire (pts (xy 610.87 375.92) (xy 630.555 375.92))
@@
     (effects (font (size 1.27 1.27)) (justify left))
   )
+  (hierarchical_label "+3.3" (shape input) (at 481.965 248.285 0) (fields_autoplaced)
+    (effects (font (size 1.27 1.27)) (justify left))
+  )
   (hierarchical_label "LED_B" (shape input) (at 574.675 278.765 0) (fields_autoplaced)
     (effects (font (size 1.27 1.27)) (justify left))
@@
         )
       )
+    )
+  )
+  (symbol (lib_id "power:+3.3V") (at 477.52 248.285 0) (mirror y) (unit 1)
+    (in_bom yes) (on_board yes) (dnp no)
+    (property "Reference" "#PWR060" (at 477.52 252.095 0)
+      (effects (font (size 1.27 1.27)) hide)
+    )
+    (property "Value" "+3.3V" (at 477.52 244.475 0)
+      (effects (font (size 1.27 1.27)))
+    )
+    (property "Footprint" "" (at 477.52 248.285 0)
+      (effects (font (size 1.27 1.27)) hide)
+    )
+    (property "Datasheet" "" (at 477.52 248.285 0)
+      (effects (font (size 1.27 1.27)) hide)
+    )
+    (pin "1")
+    (instances
+      (project "92pi"
+        (path "/6de8b922-75ab-426d-b031-f6a8fb5afbd4/2c2ae168-07bb-4d27-9d98-1a1b7c46cec2"
+          (reference "#PWR060") (unit 1)
+        )
+      )
+      (project "beepy"
+        (path "/e63e39d7-6ac0-4ffd-8aa3-1841a4541b55/832ef58d-0dd2-4973-9055-9966f4d0abfc"
+          (reference "#PWR0114") (unit 1)
+        )
+      )
